File: hardware/kinoshi-tiny-key.kicad_sch (KiCad schematic)
At the start: 97 parts, among them J1 AudioJack3, Q1 WST4041 -40V 6A, SW1 SW_SPST, SW10 SW_SPST, SW11 SW_SPST, SW12 SW_SPST, SW13 SW_SPST, SW14 SW_SPST, SW15 SW_SPST, SW16 SW_SPST, SW17 SW_SPST, SW18 SW_SPST, SW19 SW_SPST, SW2 SW_SPST, SW20 SW_SPST, SW21 SW_SPST, SW22 SW_SPST, SW23 SW_SPST, SW24 SW_SPST, SW25 SW_SPST, SW26 SW_SPST, SW27 SW_SPST, SW28 SW_SPST, SW29 SW_SPST, SW3 SW_SPST, SW30 SW_SPST, SW31 SW_SPST, SW4 SW_SPST, SW5 SW_SPST, SW6 SW_SPST, SW7 SW_SPST, SW8 SW_SPST, SW9 SW_SPST, U1 RP2040-Zero-no-bottoms, U2 74HC165, U3 74HC165, U4 74HC165, U5 74HC165

Commit message: hard: add pdfs
Other:
- company: (none) -> Kinoshita Laboratory
- title: (none) -> kinoshi tiny key 25
Changed lines of the file:
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@@
 	(generator_version "9.0")
 	(paper "A2")
+	(title_block
+		(title "kinoshi tiny key 25")
+		(date "2025-10-02")
+		(company "Kinoshita Laboratory")
+	)
 	(text "OUT"
 		(exclude_from_sim no)
