File: hardware/kinoshi-tiny-key.kicad_pcb (KiCad board)
At the start: 2 copper layers, 106 x 50 mm, 97 parts, among them J1 AudioJack3, Q1 WST4041 -40V 6A, SW1 SW_SPST, SW10 SW_SPST, SW11 SW_SPST, SW12 SW_SPST, SW13 SW_SPST, SW14 SW_SPST, SW15 SW_SPST, SW16 SW_SPST, SW17 SW_SPST, SW18 SW_SPST, SW19 SW_SPST, SW2 SW_SPST, SW20 SW_SPST, SW21 SW_SPST, SW22 SW_SPST, SW23 SW_SPST, SW24 SW_SPST, SW25 SW_SPST, SW26 SW_SPST, SW27 SW_SPST, SW28 SW_SPST, SW29 SW_SPST, SW3 SW_SPST, SW30 SW_SPST, SW31 SW_SPST, SW4 SW_SPST, SW5 SW_SPST, SW6 SW_SPST, SW7 SW_SPST, SW8 SW_SPST, SW9 SW_SPST, U1 RP2040-Zero-no-bottoms, U2 74HC165, U3 74HC165, U4 74HC165, U5 74HC165

Commit message: [hardware] update kicad version
Parts:
- D1: value LED_NeoPixel_XL-1615RGBC-WS2812B -> LED_NeoPixel_CHONGTIAN_CT-1615UGRBC/H-P6-5_C52191312; footprint my_footprint:LED_NeoPixel_XL-1615RGBC-WS2812B -> my_library:LED_NeoPixel_CHONGTIAN CT-1615UGRBCH-P6-5_C52191312
- J1: footprint my_footprint:3.5mm_Stereo_TRS_PJ-3210-4A_and_ST-005-G -> my_library:3.5mm_Stereo_TRS_PJ-3210-4A_and_ST-005-G
- LOGO1: footprint my_footprint:kinoshita-logo_simplified_300dpi -> my_library:kinoshita-logo_simplified_300dpi
- SW1, SW2, SW3, SW4, SW5, SW6: footprint my_footprint:Switch_Tactile_TS1187A26017_C22459525 -> my_library:Switch_Tactile_TS1187A26017_C22459525
- SW10, SW11, SW12, SW13, SW14, SW15, SW16, SW17, SW18, SW19, SW20, SW21, SW22, SW23, SW24, SW25, SW26, SW27, SW28, SW29, SW30, SW31, SW7, SW8, SW9: footprint my_footprint:Switch_Tactile_TSB008A2518A_C2888455 -> my_library:Switch_Tactile_TSB008A2518A_C2888455
- moved C6 1.00 mm to (77.8, 94.5)
- moved R1 0.50 mm to (79.5, 100.8)
- moved D1 0.32 mm to (78.1, 97.8), turned to 180 degrees
Connections:
- D1 pad 2: +5V -> GND
- D1 pad 3: GND -> Net-(D1-DI)
- D1 pad 4: Net-(D1-DI) -> +5V
Routing:
- net +5V: track 45.9 -> 46.4 mm
Other:
- board text added: "rev. 20260820"
